File: KiCad/robot_blance.kicad_pcb (KiCad board)
At the start: 2 copper layers, 6 parts, among them J1 Bat, U1 Esp32Dev, U2 MP1584, U3 MPU6050

Commit message: Servo
Parts:
- added D1: D, Diodes_SMD:D_0603, F.Cu at (118.1, 109.2)
- added J10: CONN_01X02, Connectors:PINHEAD1-2, F.Cu at (133.3, 113.0)
- added J11: CONN_01X03, Connectors:PINHEAD1-3, F.Cu at (148.6, 87.6)
- added J2: CONN_01X04, Connectors:Grove_1x04, F.Cu at (179.1, 87.6)
- added J3: CONN_01X04, Connectors:Grove_1x04, F.Cu at (130.8, 87.6)
- added J4: CONN_01X02, Connectors:PINHEAD1-2, F.Cu at (176.5, 113.0)
- added J5: CONN_01X02, Connectors:PINHEAD1-2, F.Cu at (179.1, 113.0)
- added J6: CONN_01X02, Connectors:PINHEAD1-2, F.Cu at (181.6, 113.0)
- added J7: CONN_01X03, Connectors:PINHEAD1-3, F.Cu at (165.1, 87.6)
- added J8: CONN_01X02, Connectors:PINHEAD1-2, F.Cu at (128.3, 113.0)
- added J9: CONN_01X02, Connectors:PINHEAD1-2, F.Cu at (130.8, 113.0)
- added R1: R, Resistors_THT:R_Axial_DIN0204_L3.6mm_D1.6mm_P5.08mm_Horizontal, F.Cu at (115.6, 114.3)
- added R2: R, Resistors_THT:R_Axial_DIN0204_L3.6mm_D1.6mm_P5.08mm_Horizontal, F.Cu at (115.6, 120.7)
- moved DRV1 5.39 mm to (184.2, 101.6)
- moved U3 5.39 mm to (168.9, 110.5)
- moved DRV2 5.39 mm to (135.9, 101.6)
- moved J1 3.81 mm to (116.8, 100.3)
- moved U1 3.81 mm to (168.9, 134.6)
- moved U2 3.81 mm to (124.5, 134.6)
Connections:
- DRV1 pad 1: (no net) -> Net-(DRV1-Pad1)
- DRV1 pad 10: (no net) -> Net-(DRV1-Pad10)
- DRV1 pad 11: (no net) -> Net-(DRV1-Pad11)
- DRV1 pad 12: (no net) -> Net-(DRV1-Pad12)
- DRV1 pad 13: (no net) -> Net-(DRV1-Pad13)
- DRV1 pad 14: (no net) -> Net-(DRV1-Pad14)
- DRV1 pad 15: (no net) -> Net-(C1-Pad2)
- DRV1 pad 16: (no net) -> Net-(C1-Pad1)
- DRV1 pad 2: (no net) -> Net-(DRV1-Pad2)
- DRV1 pad 3: (no net) -> Net-(DRV1-Pad3)
- DRV1 pad 4: (no net) -> Net-(DRV1-Pad4)
- DRV1 pad 5: (no net) -> Net-(DRV1-Pad5)
- DRV1 pad 6: (no net) -> Net-(DRV1-Pad5)
- DRV1 pad 7: (no net) -> Net-(DRV1-Pad7)
- DRV1 pad 8: (no net) -> Net-(DRV1-Pad8)
- DRV1 pad 9: (no net) -> Net-(C1-Pad2)
- DRV2 pad 1: (no net) -> Net-(DRV2-Pad1)
- DRV2 pad 10: (no net) -> Net-(DRV1-Pad10)
- DRV2 pad 11: (no net) -> Net-(DRV2-Pad11)
- DRV2 pad 12: (no net) -> Net-(DRV2-Pad12)
- DRV2 pad 13: (no net) -> Net-(DRV2-Pad13)
- DRV2 pad 14: (no net) -> Net-(DRV2-Pad14)
- DRV2 pad 15: (no net) -> Net-(C1-Pad2)
- DRV2 pad 16: (no net) -> Net-(C1-Pad1)
- DRV2 pad 2: (no net) -> Net-(DRV2-Pad2)
- DRV2 pad 3: (no net) -> Net-(DRV2-Pad3)
- DRV2 pad 4: (no net) -> Net-(DRV2-Pad4)
- DRV2 pad 5: (no net) -> Net-(DRV2-Pad5)
- DRV2 pad 6: (no net) -> Net-(DRV2-Pad5)
- DRV2 pad 7: (no net) -> Net-(DRV2-Pad7)
- DRV2 pad 8: (no net) -> Net-(DRV2-Pad8)
- DRV2 pad 9: (no net) -> Net-(C1-Pad2)
- J1 pad 1: (no net) -> +12V
- J1 pad 2: Net-(J1-Pad2) -> GND
- U1 pad 1: (no net) -> Net-(DRV1-Pad10)
- U1 pad 10: (no net) -> Net-(U1-Pad10)
- U1 pad 11: (no net) -> Net-(U1-Pad11)
- U1 pad 12: (no net) -> Net-(U1-Pad12)
- U1 pad 13: (no net) -> Net-(R1-Pad2)
- U1 pad 14: (no net) -> Net-(U1-Pad14)
- U1 pad 15: (no net) -> Net-(U1-Pad15)
- U1 pad 16: (no net) -> Net-(DRV1-Pad7)
- U1 pad 17: (no net) -> Net-(DRV1-Pad8)
- U1 pad 18: (no net) -> Net-(U1-Pad18)
- U1 pad 19: (no net) -> Net-(U1-Pad19)
- U1 pad 2: (no net) -> Net-(U1-Pad2)
- U1 pad 20: (no net) -> Net-(U1-Pad20)
- U1 pad 21: (no net) -> Net-(U1-Pad21)
- U1 pad 22: (no net) -> Net-(U1-Pad22)
- U1 pad 23: (no net) -> Net-(U1-Pad23)
- U1 pad 24: (no net) -> Net-(U1-Pad24)
- U1 pad 25: (no net) -> Net-(U1-Pad25)
- U1 pad 26: (no net) -> Net-(U1-Pad26)
- U1 pad 27: (no net) -> Net-(U1-Pad27)
- U1 pad 28: (no net) -> Net-(U1-Pad28)
- U1 pad 29: (no net) -> Net-(U1-Pad29)
- U1 pad 3: (no net) -> Net-(U1-Pad3)
- U1 pad 30: (no net) -> Net-(U1-Pad30)
- U1 pad 31: (no net) -> Net-(U1-Pad31)
- U1 pad 32: (no net) -> Net-(DRV2-Pad8)
- U1 pad 33: (no net) -> Net-(U1-Pad33)
- U1 pad 34: (no net) -> Net-(DRV2-Pad7)
- U1 pad 35: (no net) -> Net-(U1-Pad35)
- U1 pad 36: (no net) -> Net-(J11-Pad1)
- U1 pad 37: (no net) -> Net-(J7-Pad1)
- U1 pad 38: (no net) -> Net-(U1-Pad38)
- U1 pad 4: (no net) -> Net-(U1-Pad4)
- U1 pad 5: (no net) -> Net-(U1-Pad5)
- U1 pad 6: Net-(U1-Pad6) -> Net-(C1-Pad2)
- U1 pad 7: (no net) -> Net-(U1-Pad7)
- U1 pad 8: (no net) -> Net-(U1-Pad8)
- U1 pad 9: (no net) -> Net-(U1-Pad9)
- U2 pad 2: Net-(J1-Pad2) -> Net-(U2-Pad2)
- U2 pad 3: Net-(U1-Pad6) -> Net-(U2-Pad3)
- U3 pad 1: (no net) -> Net-(DRV1-Pad10)
- U3 pad 2: (no net) -> Net-(U3-Pad2)
- U3 pad 3: (no net) -> Net-(U1-Pad22)
- U3 pad 4: (no net) -> Net-(U1-Pad25)
- U3 pad 5: (no net) -> Net-(U3-Pad5)
- U3 pad 6: (no net) -> Net-(U3-Pad6)
- U3 pad 7: (no net) -> Net-(U3-Pad7)
- U3 pad 8: (no net) -> Net-(U3-Pad8)

Commit message: Router
Parts:
- added C1: CP1, Capacitors_THT:CP_Radial_D10.0mm_P3.50mm, F.Cu at (147.3, 114.3)
- added C2: CP1, Capacitors_THT:CP_Radial_D10.0mm_P3.50mm, F.Cu at (124.5, 114.3)
- D1: footprint Diodes_SMD:D_0603 -> Diodes_THT:D_DO-41_SOD81_P5.08mm_Vertical_AnodeUp
- J1: moved to B.Cu
- moved J1 52.8 mm to (125.7, 152.4), turned to 180 degrees
- moved U3 39.4 mm to (168.9, 149.9)
- moved D1 35.4 mm to (127.0, 143.5), turned to 180 degrees
- moved J6 31.2 mm to (153.7, 127.0)
- moved DRV1 31.2 mm to (156.2, 115.6)
- moved J4 31.2 mm to (148.6, 127.0)
- moved J5 31.2 mm to (151.1, 127.0)
- moved J2 27.5 mm to (156.2, 102.9)
- moved R1 25.0 mm to (121.9, 138.4)
- moved J7 24.4 mm to (146.1, 102.9)
- moved U1 21.0 mm to (188.0, 125.7), turned to 180 degrees
- moved J11 19.8 mm to (135.9, 102.9)
- moved U2 17.3 mm to (138.4, 144.8)
- moved J3 16.5 mm to (124.5, 102.9)
- moved R2 15.3 mm to (121.9, 134.6)
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Connections:
- DRV1 pad 1: Net-(DRV1-Pad1) -> (no net)
- DRV1 pad 15: Net-(C1-Pad2) -> GND
- DRV1 pad 9: Net-(C1-Pad2) -> GND
- DRV2 pad 1: Net-(DRV2-Pad1) -> (no net)
- DRV2 pad 15: Net-(C1-Pad2) -> GND
- DRV2 pad 9: Net-(C1-Pad2) -> GND
- J11 pad 3: Net-(C1-Pad2) -> GND
- J7 pad 3: Net-(C1-Pad2) -> GND
- U1 pad 10: Net-(U1-Pad10) -> (no net)
- U1 pad 11: Net-(U1-Pad11) -> (no net)
- U1 pad 12: Net-(U1-Pad12) -> (no net)
- U1 pad 14: Net-(U1-Pad14) -> (no net)
- U1 pad 15: Net-(U1-Pad15) -> (no net)
- U1 pad 18: Net-(U1-Pad18) -> (no net)
- U1 pad 19: Net-(U1-Pad19) -> (no net)
- U1 pad 2: Net-(U1-Pad2) -> (no net)
- U1 pad 20: Net-(U1-Pad20) -> (no net)
- U1 pad 21: Net-(U1-Pad21) -> (no net)
- U1 pad 23: Net-(U1-Pad23) -> (no net)
- U1 pad 24: Net-(U1-Pad24) -> (no net)
- U1 pad 26: Net-(U1-Pad26) -> (no net)
- U1 pad 27: Net-(U1-Pad27) -> (no net)
- U1 pad 28: Net-(U1-Pad28) -> (no net)
- U1 pad 29: Net-(U1-Pad29) -> (no net)
- U1 pad 3: Net-(U1-Pad3) -> (no net)
- U1 pad 30: Net-(U1-Pad30) -> (no net)
- U1 pad 31: Net-(U1-Pad31) -> (no net)
- U1 pad 33: Net-(U1-Pad33) -> (no net)
- U1 pad 35: Net-(U1-Pad35) -> (no net)
- U1 pad 38: Net-(U1-Pad38) -> (no net)
- U1 pad 4: Net-(U1-Pad4) -> (no net)
- U1 pad 5: Net-(U1-Pad5) -> (no net)
- U1 pad 6: Net-(C1-Pad2) -> GND
- U1 pad 7: Net-(U1-Pad7) -> (no net)
- U1 pad 8: Net-(U1-Pad8) -> (no net)
- U1 pad 9: Net-(U1-Pad9) -> (no net)
- U2 pad 1: Net-(U2-Pad1) -> Net-(C1-Pad1)
- U2 pad 2: Net-(U2-Pad2) -> GND
- U2 pad 3: Net-(U2-Pad3) -> GND
- U2 pad 4: Net-(U2-Pad4) -> Net-(DRV1-Pad10)
- U3 pad 2: Net-(U3-Pad2) -> GND
- U3 pad 5: Net-(U3-Pad5) -> (no net)
- U3 pad 6: Net-(U3-Pad6) -> (no net)
- U3 pad 7: Net-(U3-Pad7) -> (no net)
- U3 pad 8: Net-(U3-Pad8) -> (no net)
Routing:
- net Net-(R1-Pad2): track 0.00 -> 123.1 mm
- net Net-(J11-Pad1): track 0.00 -> 62.4 mm
- net Net-(C1-Pad1): track 0.00 -> 62.1 mm
- net Net-(J7-Pad1): track 0.00 -> 41.8 mm
- net GND: track 0.00 -> 37.1 mm
- net Net-(DRV1-Pad10): track 0.00 -> 28.5 mm
- net Net-(U1-Pad22): track 0.00 -> 24.2 mm
- net Net-(U1-Pad25): track 0.00 -> 21.1 mm
- net Net-(DRV2-Pad11): track 0.00 -> 9.87 mm
- net Net-(DRV1-Pad14): track 0.00 -> 9.72 mm
- net Net-(DRV2-Pad12): track 0.00 -> 9.65 mm
- net Net-(DRV1-Pad13): track 0.00 -> 9.50 mm
- net Net-(DRV2-Pad13): track 0.00 -> 9.42 mm
- net +12V: track 0.00 -> 9.42 mm
- net Net-(DRV1-Pad12): track 0.00 -> 9.28 mm
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- added copper zone on F.Cu, net GND

Commit message: router
Connections:
- J10 pad 2: Net-(J10-Pad2) -> Net-(DRV1-Pad10)
- J8 pad 2: Net-(J10-Pad2) -> Net-(DRV1-Pad10)
- J9 pad 2: Net-(J10-Pad2) -> Net-(DRV1-Pad10)
Routing:
- net Net-(DRV1-Pad10): track 28.5 -> 134.8 mm
- net Net-(DRV2-Pad4): track 0.00 -> 3.81 mm
- net Net-(DRV2-Pad3): track 0.00 -> 3.81 mm
- net Net-(DRV2-Pad2): track 0.00 -> 3.81 mm
- net Net-(DRV1-Pad4): track 0.00 -> 3.81 mm
- net Net-(DRV1-Pad3): track 0.00 -> 3.81 mm
- net Net-(DRV1-Pad2): track 0.00 -> 3.81 mm
- net Net-(DRV2-Pad5): track 0.00 -> 2.54 mm
- net Net-(DRV1-Pad5): track 0.00 -> 2.54 mm
Changed lines of the file:
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@@
 (kicad_pcb (version 4) (host pcbnew 4.0.6)
   (general
-    (links 61)
-    (no_connects 23)
+    (links 62)
+    (no_connects 19)
     (area 0 0 0 0)
     (thickness 1.6)
     (drawings 9)
-    (tracks 91)
+    (tracks 124)
     (zones 0)
     (modules 21)
-    (nets 31)
+    (nets 30)
   )
   (page A4)
@@
   (net 27 "Net-(C1-Pad1)")
   (net 28 "Net-(J7-Pad1)")
-  (net 29 "Net-(J10-Pad2)")
-  (net 30 "Net-(J11-Pad1)")
+  (net 29 "Net-(J11-Pad1)")
   (net_class Default "This is the default net class."
     (clearance 0.2)
@@
     (add_net "Net-(DRV2-Pad7)")
     (add_net "Net-(DRV2-Pad8)")
-    (add_net "Net-(J10-Pad2)")
     (add_net "Net-(J11-Pad1)")
     (add_net "Net-(J7-Pad1)")
@@
     (pad 35 thru_hole circle (at 13.97 11.43 180) (size 1.524 1.524) (drill 0.762) (layers *.Cu *.Mask))
     (pad 36 thru_hole circle (at 13.97 13.97 180) (size 1.524 1.524) (drill 0.762) (layers *.Cu *.Mask)
-      (net 30 "Net-(J11-Pad1)"))
+      (net 29 "Net-(J11-Pad1)"))
     (pad 37 thru_hole circle (at 13.97 16.51 180) (size 1.524 1.524) (drill 0.762) (layers *.Cu *.Mask)
       (net 28 "Net-(J7-Pad1)"))
@@
       (net 12 "Net-(DRV2-Pad2)"))
     (pad 2 thru_hole circle (at 2.54 0 270) (size 1.51 1.51) (drill 1) (layers *.Cu *.Mask)
-      (net 29 "Net-(J10-Pad2)"))
+      (net 7 "Net-(DRV1-Pad10)"))
   )
   (module Connectors:PINHEAD1-2 (layer F.Cu)
@@
       (net 13 "Net-(DRV2-Pad3)"))
     (pad 2 thru_hole circle (at 2.54 0 270) (size 1.51 1.51) (drill 1) (layers *.Cu *.Mask)
-      (net 29 "Net-(J10-Pad2)"))
+      (net 7 "Net-(DRV1-Pad10)"))
   )
   (module Connectors:PINHEAD1-2 (layer F.Cu)
@@
       (net 14 "Net-(DRV2-Pad4)"))
     (pad 2 thru_hole circle (at 2.54 0 270) (size 1.51 1.51) (drill 1) (layers *.Cu *.Mask)
-      (net 29 "Net-(J10-Pad2)"))
+      (net 7 "Net-(DRV1-Pad10)"))
   )
   (module Connectors:PINHEAD1-3 (layer F.Cu)
@@
     (fp_line (start 6.6 3.42) (end -1.52 3.42) (layer F.CrtYd) (width 0.05))
     (pad 1 thru_hole oval (at 0 0) (size 1.51 3.01) (drill 1) (layers *.Cu *.Mask)
-      (net 30 "Net-(J11-Pad1)"))
+      (net 29 "Net-(J11-Pad1)"))
     (pad 2 thru_hole oval (at 2.54 0) (size 1.51 3.01) (drill 1) (layers *.Cu *.Mask)
       (net 7 "Net-(DRV1-Pad10)"))
@@
   (gr_circle (center 168.91 153.67) (end 170.18 153.67) (layer F.Adhes) (width 0.2))
   (gr_circle (center 168.91 105.41) (end 170.18 105.41) (layer F.Adhes) (width 0.2))
-  (segment (start 134.366 154.051) (end 131.826 154.051) (width 0.25) (layer F.Cu) (net 7) (status C00000))
-  (segment (start 134.366 154.051) (end 134.366 155.956) (width 0.25) (layer F.Cu) (net 7) (status 400000))
-  (segment (start 150.11 154.69) (end 150.11 148.16) (width 0.25) (layer F.Cu) (net 7) (status 800000))
+  (segment (start 148.59 127) (end 148.59 123.19) (width 0.25) (layer F.Cu) (net 1))
+  (segment (start 151.13 127) (end 151.13 123.19) (width 0.25) (layer F.Cu) (net 2))
+  (segment (start 153.67 127) (end 153.67 123.19) (width 0.25) (layer F.Cu) (net 3))
+  (segment (start 158.75 123.19) (end 156.21 123.19) (width 0.25) (layer F.Cu) (net 4) (status C00000))
+  (segment (start 161.29 110.49) (end 161.29 109.22) (width 0.25) (layer F.Cu) (net 7) (status 400000))
+  (segment (start 148.59 100.33) (end 148.59 102.87) (width 0.25) (layer F.Cu) (net 7) (status 800000))
+  (segment (start 149.86 99.06) (end 148.59 100.33) (width 0.25) (layer F.Cu) (net 7))
+  (segment (start 165.1 99.06) (end 149.86 99.06) (width 0.25) (layer F.Cu) (net 7))
+  (segment (start 166.37 100.33) (end 165.1 99.06) (width 0.25) (layer F.Cu) (net 7))
+  (segment (start 166.37 101.6) (end 166.37 100.33) (width 0.25) (layer F.Cu) (net 7))
+  (segment (start 166.37 105.41) (end 166.37 101.6) (width 0.25) (layer F.Cu) (net 7))
+  (segment (start 165.1 106.68) (end 166.37 105.41) (width 0.25) (layer F.Cu) (net 7))
+  (segment (start 163.83 106.68) (end 165.1 106.68) (width 0.25) (layer F.Cu) (net 7))
+  (segment (start 161.29 109.22) (end 163.83 106.68) (width 0.25) (layer F.Cu) (net 7))
+  (segment (start 138.43 110.49) (end 138.43 109.22) (width 0.25) (layer F.Cu) (net 7) (status 400000))
+  (segment (start 148.59 106.68) (end 148.59 102.87) (width 0.25) (layer F.Cu) (net 7) (status 800000))
+  (segment (start 147.32 107.95) (end 148.59 106.68) (width 0.25) (layer F.Cu) (net 7))
+  (segment (start 139.7 107.95) (end 147.32 107.95) (width 0.25) (layer F.Cu) (net 7))
+  (segment (start 138.43 109.22) (end 139.7 107.95) (width 0.25) (layer F.Cu) (net 7))
+  (segment (start 138.43 110.49) (end 138.43 102.87) (width 0.25) (layer F.Cu) (net 7) (status C00000))
+  (segment (start 130.81 129.54) (end 148.59 129.54) (width 0.25) (layer F.Cu) (net 7) (status 400000))
+  (segment (start 151.13 129.54) (end 148.59 129.54) (width 0.25) (layer F.Cu) (net 7))
+  (segment (start 151.13 129.54) (end 153.67 129.54) (width 0.25) (layer F.Cu) (net 7))
+  (segment (start 150.11 148.16) (end 150.11 134.37) (width 0.25) (layer F.Cu) (net 7))
+  (segment (start 151.13 132.08) (end 148.59 129.54) (width 0.25) (layer F.Cu) (net 7))
+  (segment (start 151.13 133.35) (end 151.13 132.08) (width 0.25) (layer F.Cu) (net 7))
+  (segment (start 150.11 134.37) (end 151.13 133.35) (width 0.25) (layer F.Cu) (net 7))
+  (segment (start 134.366 154.051) (end 131.826 154.051) (width 0.25) (layer F.Cu) (net 7))
+  (segment (start 134.366 154.051) (end 134.366 155.956) (width 0.25) (layer F.Cu) (net 7))
+  (segment (start 150.11 154.69) (end 150.11 148.16) (width 0.25) (layer F.Cu) (net 7))
   (segment (start 147.32 157.48) (end 150.11 154.69) (width 0.25) (layer F.Cu) (net 7))
   (segment (start 135.89 157.48) (end 147.32 157.48) (width 0.25) (layer F.Cu) (net 7))
   (segment (start 134.366 155.956) (end 135.89 157.48) (width 0.25) (layer F.Cu) (net 7))
+  (segment (start 128.27 129.54) (end 130.81 129.54) (width 0.25) (layer F.Cu) (net 7))
+  (segment (start 125.73 129.54) (end 128.27 129.54) (width 0.25) (layer F.Cu) (net 7))
   (segment (start 158.75 110.49) (end 158.75 109.22) (width 0.25) (layer F.Cu) (net 8))
   (segment (start 162.21 105.76) (end 162.21 102.87) (width 0.25) (layer F.Cu) (net 8))
@@
   (segment (start 151.13 109.22) (end 156.21 104.14) (width 0.25) (layer F.Cu) (net 11))
   (segment (start 151.13 109.22) (end 151.13 110.49) (width 0.25) (layer F.Cu) (net 11))
+  (segment (start 125.73 127) (end 125.73 123.19) (width 0.25) (layer F.Cu) (net 12))
+  (segment (start 128.27 127) (end 128.27 123.19) (width 0.25) (layer F.Cu) (net 13))
+  (segment (start 130.81 127) (end 130.81 123.19) (width 0.25) (layer F.Cu) (net 14))
+  (segment (start 135.89 123.19) (end 133.35 123.19) (width 0.25) (layer F.Cu) (net 15) (status C00000))
   (segment (start 135.89 110.49) (end 135.89 109.22) (width 0.25) (layer F.Cu) (net 18))
   (segment (start 130.81 104.14) (end 130.81 103.22) (width 0.25) (layer F.Cu) (net 18))
@@
   (segment (start 163.83 139.7) (end 173.99 139.7) (width 0.25) (layer F.Cu) (net 26))
   (segment (start 157.73 145.8) (end 163.83 139.7) (width 0.25) (layer F.Cu) (net 26))
-  (segment (start 131.826 135.509) (end 134.366 135.509) (width 0.25) (layer F.Cu) (net 27) (status C00000))
-  (segment (start 131.826 135.509) (end 131.826 133.096) (width 0.25) (layer F.Cu) (net 27) (status 400000))
+  (segment (start 131.826 135.509) (end 134.366 135.509) (width 0.25) (layer F.Cu) (net 27))
+  (segment (start 131.826 135.509) (end 131.826 133.096) (width 0.25) (layer F.Cu) (net 27))
   (segment (start 130.81 132.08) (end 119.38 132.08) (width 0.25) (layer F.Cu) (net 27))
   (segment (start 131.826 133.096) (end 130.81 132.08) (width 0.25) (layer F.Cu) (net 27))
@@
   (segment (start 171.45 107.95) (end 171.45 101.6) (width 0.25) (layer F.Cu) (net 28))
   (segment (start 172.72 109.22) (end 171.45 107.95) (width 0.25) (layer F.Cu) (net 28))
-  (segment (start 173.99 111.76) (end 176.53 109.22) (width 0.25) (layer F.Cu) (net 30))
-  (segment (start 135.89 99.06) (end 135.89 102.87) (width 0.25) (layer F.Cu) (net 30))
-  (segment (start 139.7 95.25) (end 135.89 99.06) (width 0.25) (layer F.Cu) (net 30))
-  (segment (start 172.72 95.25) (end 139.7 95.25) (width 0.25) (layer F.Cu) (net 30))
-  (segment (start 177.8 100.33) (end 172.72 95.25) (width 0.25) (layer F.Cu) (net 30))
-  (segment (start 177.8 107.95) (end 177.8 100.33) (width 0.25) (layer F.Cu) (net 30))
-  (segment (start 176.53 109.22) (end 177.8 107.95) (width 0.25) (layer F.Cu) (net 30))
+  (segment (start 173.99 111.76) (end 176.53 109.22) (width 0.25) (layer F.Cu) (net 29))
+  (segment (start 135.89 99.06) (end 135.89 102.87) (width 0.25) (layer F.Cu) (net 29))
+  (segment (start 139.7 95.25) (end 135.89 99.06) (width 0.25) (layer F.Cu) (net 29))
+  (segment (start 172.72 95.25) (end 139.7 95.25) (width 0.25) (layer F.Cu) (net 29))
+  (segment (start 177.8 100.33) (end 172.72 95.25) (width 0.25) (layer F.Cu) (net 29))
+  (segment (start 177.8 107.95) (end 177.8 100.33) (width 0.25) (layer F.Cu) (net 29))
+  (segment (start 176.53 109.22) (end 177.8 107.95) (width 0.25) (layer F.Cu) (net 29))
   (zone (net 23) (net_name GND) (layer F.Cu) (hatch edge 0.508)
     (connect_pads (clearance 0.508))
     (min_thickness 0.254)
-    (fill yes (arc_segments 16) (thermal_gap 0.508) (thermal_bridge_width 0.508))
+    (fill (arc_segments 16) (thermal_gap 0.508) (thermal_bridge_width 0.508))
     (polygon
       (pts
