File: KiCad/robot_blance.kicad_pcb (KiCad board)
At the start: 2 copper layers, 21 parts, among them J1 Bat, J10 CONN_01X02, J11 CONN_01X03, J2 CONN_01X04, J3 CONN_01X04, J4 CONN_01X02, J5 CONN_01X02, J6 CONN_01X02, J7 CONN_01X03, J8 CONN_01X02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

Commit message: Net
Routing:
- net +5V: track 134.8 -> 303.3 mm
- net Net-(D1-Pad2): track 48.1 -> 13.6 mm
- net +12V: track 23.5 -> 57.9 mm
Other:
- board outline added: 91.4 x 71.1 mm
- net class Default: trace_width 0.25 -> 1
Changed lines of the file:
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@@
   (general
     (links 62)
-    (no_connects 20)
+    (no_connects 19)
     (area 0 0 0 0)
     (thickness 1.6)
-    (drawings 9)
-    (tracks 124)
+    (drawings 13)
+    (tracks 145)
     (zones 0)
     (modules 21)
@@
   )
   (setup
-    (last_trace_width 0.25)
+    (last_trace_width 1)
     (trace_clearance 0.2)
     (zone_clearance 0.508)
@@
   (net_class Default "This is the default net class."
     (clearance 0.2)
-    (trace_width 0.25)
+    (trace_width 1)
     (via_dia 0.6)
     (via_drill 0.4)
@@
     )
   )
+  (gr_line (start 114.3 162.56) (end 114.3 91.44) (angle 90) (layer Edge.Cuts) (width 0.15))
+  (gr_line (start 205.74 162.56) (end 114.3 162.56) (angle 90) (layer Edge.Cuts) (width 0.15))
+  (gr_line (start 205.74 91.44) (end 205.74 162.56) (angle 90) (layer Edge.Cuts) (width 0.15))
+  (gr_line (start 114.3 91.44) (end 205.74 91.44) (angle 90) (layer Edge.Cuts) (width 0.15))
   (gr_circle (center 118.11 110.49) (end 119.38 110.49) (layer F.Adhes) (width 0.2))
   (gr_line (start 205.74 162.56) (end 205.74 91.44) (angle 90) (layer F.Adhes) (width 0.2))
@@
   (segment (start 124.46 111.76) (end 123.19 110.49) (width 0.25) (layer F.Cu) (net 21))
   (segment (start 119.38 114.3) (end 123.19 110.49) (width 0.25) (layer F.Cu) (net 21))
+  (segment (start 119.38 132.08) (end 119.38 114.3) (width 0.25) (layer F.Cu) (net 21))
+  (segment (start 130.81 132.08) (end 119.38 132.08) (width 0.25) (layer F.Cu) (net 21))
+  (segment (start 119.38 135.89) (end 119.38 132.08) (width 0.25) (layer F.Cu) (net 21))
+  (segment (start 131.826 133.096) (end 130.81 132.08) (width 0.25) (layer F.Cu) (net 21))
   (segment (start 123.19 152.4) (end 123.19 148.59) (width 0.25) (layer F.Cu) (net 22))
   (segment (start 124.46 137.16) (end 121.92 134.62) (width 0.25) (layer F.Cu) (net 22))
@@
   (segment (start 131.826 135.509) (end 134.366 135.509) (width 0.25) (layer F.Cu) (net 28))
   (segment (start 131.826 135.509) (end 131.826 133.096) (width 0.25) (layer F.Cu) (net 28))
-  (segment (start 130.81 132.08) (end 119.38 132.08) (width 0.25) (layer F.Cu) (net 28))
-  (segment (start 131.826 133.096) (end 130.81 132.08) (width 0.25) (layer F.Cu) (net 28))
-  (segment (start 119.38 135.89) (end 119.38 132.08) (width 0.25) (layer F.Cu) (net 28))
-  (segment (start 119.38 132.08) (end 119.38 114.3) (width 0.25) (layer F.Cu) (net 28))
   (segment (start 121.92 138.43) (end 119.38 135.89) (width 0.25) (layer F.Cu) (net 28))
   (segment (start 121.92 143.51) (end 121.92 138.43) (width 0.25) (layer F.Cu) (net 28))
+  (segment (start 143.51 120.65) (end 151.13 120.65) (width 1) (layer F.Cu) (net 29))
+  (segment (start 151.13 120.65) (end 156.21 115.57) (width 1) (layer F.Cu) (net 29))
+  (segment (start 156.21 115.57) (end 158.75 115.57) (width 1) (layer F.Cu) (net 29))
+  (segment (start 158.75 115.57) (end 161.29 113.03) (width 1) (layer F.Cu) (net 29))
+  (segment (start 161.29 113.03) (end 161.29 110.49) (width 1) (layer F.Cu) (net 29))
+  (segment (start 201.93 106.68) (end 193.04 106.68) (width 1) (layer F.Cu) (net 29))
+  (segment (start 150.11 153.92) (end 150.11 148.16) (width 1) (layer F.Cu) (net 29))
+  (segment (start 153.67 157.48) (end 150.11 153.92) (width 1) (layer F.Cu) (net 29))
+  (segment (start 181.61 157.48) (end 153.67 157.48) (width 1) (layer F.Cu) (net 29))
+  (segment (start 187.96 151.13) (end 181.61 157.48) (width 1) (layer F.Cu) (net 29))
+  (segment (start 187.96 111.76) (end 187.96 151.13) (width 1) (layer F.Cu) (net 29))
+  (segment (start 193.04 106.68) (end 187.96 111.76) (width 1) (layer F.Cu) (net 29))
+  (segment (start 143.51 121.92) (end 143.51 120.65) (width 1) (layer F.Cu) (net 29))
+  (segment (start 138.43 110.49) (end 138.43 111.76) (width 1) (layer F.Cu) (net 29))
+  (segment (start 138.43 111.76) (end 143.51 116.84) (width 1) (layer F.Cu) (net 29))
+  (segment (start 143.51 116.84) (end 143.51 120.65) (width 1) (layer F.Cu) (net 29))
+  (segment (start 130.81 129.54) (end 138.43 129.54) (width 1) (layer F.Cu) (net 29))
+  (segment (start 143.51 116.84) (end 138.43 111.76) (width 1) (layer F.Cu) (net 29))
+  (segment (start 143.51 124.46) (end 143.51 121.92) (width 1) (layer F.Cu) (net 29))
+  (segment (start 143.51 120.65) (end 143.51 116.84) (width 1) (layer F.Cu) (net 29))
+  (segment (start 138.43 129.54) (end 143.51 124.46) (width 1) (layer F.Cu) (net 29))
   (segment (start 161.29 110.49) (end 161.29 109.22) (width 0.25) (layer F.Cu) (net 29))
+  (segment (start 161.29 109.22) (end 163.83 106.68) (width 0.25) (layer F.Cu) (net 29))
+  (segment (start 163.83 106.68) (end 165.1 106.68) (width 0.25) (layer F.Cu) (net 29))
+  (segment (start 165.1 106.68) (end 166.37 105.41) (width 0.25) (layer F.Cu) (net 29))
+  (segment (start 166.37 105.41) (end 166.37 101.6) (width 0.25) (layer F.Cu) (net 29))
+  (segment (start 166.37 101.6) (end 166.37 100.33) (width 0.25) (layer F.Cu) (net 29))
+  (segment (start 166.37 100.33) (end 165.1 99.06) (width 0.25) (layer F.Cu) (net 29))
+  (segment (start 165.1 99.06) (end 149.86 99.06) (width 0.25) (layer F.Cu) (net 29))
+  (segment (start 149.86 99.06) (end 148.59 100.33) (width 0.25) (layer F.Cu) (net 29))
   (segment (start 148.59 100.33) (end 148.59 102.87) (width 0.25) (layer F.Cu) (net 29))
-  (segment (start 149.86 99.06) (end 148.59 100.33) (width 0.25) (layer F.Cu) (net 29))
-  (segment (start 165.1 99.06) (end 149.86 99.06) (width 0.25) (layer F.Cu) (net 29))
-  (segment (start 166.37 100.33) (end 165.1 99.06) (width 0.25) (layer F.Cu) (net 29))
-  (segment (start 166.37 101.6) (end 166.37 100.33) (width 0.25) (layer F.Cu) (net 29))
-  (segment (start 166.37 105.41) (end 166.37 101.6) (width 0.25) (layer F.Cu) (net 29))
-  (segment (start 165.1 106.68) (end 166.37 105.41) (width 0.25) (layer F.Cu) (net 29))
-  (segment (start 163.83 106.68) (end 165.1 106.68) (width 0.25) (layer F.Cu) (net 29))
-  (segment (start 161.29 109.22) (end 163.83 106.68) (width 0.25) (layer F.Cu) (net 29))
   (segment (start 138.43 110.49) (end 138.43 109.22) (width 0.25) (layer F.Cu) (net 29))
+  (segment (start 138.43 109.22) (end 139.7 107.95) (width 0.25) (layer F.Cu) (net 29))
+  (segment (start 139.7 107.95) (end 147.32 107.95) (width 0.25) (layer F.Cu) (net 29))
+  (segment (start 147.32 107.95) (end 148.59 106.68) (width 0.25) (layer F.Cu) (net 29))
   (segment (start 148.59 106.68) (end 148.59 102.87) (width 0.25) (layer F.Cu) (net 29))
-  (segment (start 147.32 107.95) (end 148.59 106.68) (width 0.25) (layer F.Cu) (net 29))
-  (segment (start 139.7 107.95) (end 147.32 107.95) (width 0.25) (layer F.Cu) (net 29))
-  (segment (start 138.43 109.22) (end 139.7 107.95) (width 0.25) (layer F.Cu) (net 29))
   (segment (start 138.43 110.49) (end 138.43 102.87) (width 0.25) (layer F.Cu) (net 29))
   (segment (start 130.81 129.54) (end 148.59 129.54) (width 0.25) (layer F.Cu) (net 29))
@@
     (polygon
       (pts
-        (xy 205.74 162.56) (xy 114.3 162.56) (xy 114.3 91.44) (xy 205.74 91.44) (xy 205.74 162.56)
+        (xy 205.74 162.56) (xy 114.3 162.56) (xy 114.3 91.44) (xy 205.74 91.44)
       )
     )

Commit message: Net
Parts:
- moved C1 1.27 mm to (147.3, 113.0)
- moved C2 1.27 mm to (124.5, 113.0)
Connections:
- C1 pad 1: +12V -> Net-(C1-Pad1)
- C2 pad 1: +12V -> Net-(C1-Pad1)
- D1 pad 2: Net-(D1-Pad2) -> Net-(C1-Pad1)
- DRV1 pad 16: +12V -> Net-(C1-Pad1)
- DRV2 pad 16: +12V -> Net-(C1-Pad1)
- R1 pad 1: Net-(D1-Pad2) -> Net-(C1-Pad1)
- U1 pad 20: (no net) -> GND
- U2 pad 1: Net-(D1-Pad2) -> Net-(C1-Pad1)
Routing:
- net Net-(R1-Pad2): track 123.1 -> 3.81 mm
- net Net-(C1-Pad1): track 0.00 -> 86.6 mm
- net Net-(J11-Pad1): track 62.4 -> 0.00 mm
- net Net-(J7-Pad1): track 41.8 -> 0.00 mm
- net +12V: track 57.9 -> 16.3 mm
- net Net-(DRV2-Pad7): track 0.00 -> 39.7 mm
- net GND: track 37.1 -> 0.00 mm
- net Net-(DRV2-Pad8): track 0.00 -> 36.1 mm
- net +5V: track 303.3 -> 317.0 mm
- net Net-(D1-Pad2): track 13.6 -> 0.00 mm
- net Net-(DRV1-Pad14): track 9.72 -> 0.00 mm
- net Net-(DRV2-Pad12): track 9.65 -> 0.00 mm
- net Net-(DRV1-Pad13): track 9.50 -> 0.00 mm
- net Net-(DRV2-Pad13): track 9.42 -> 0.00 mm
- net Net-(DRV2-Pad11): track 9.87 -> 0.49 mm
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Other:
- net class Default: trace_width 1 -> 0.5

Commit message: Net
Routing:
- net Net-(R1-Pad2): track 3.81 -> 127.1 mm
- net Net-(J11-Pad1): track 0.00 -> 82.7 mm, vias 0 -> 2
- net Net-(J7-Pad1): track 0.00 -> 64.6 mm, vias 0 -> 2
- net +5V: track 317.0 -> 298.8 mm
- net Net-(DRV2-Pad12): track 0.00 -> 10.5 mm
- net Net-(DRV2-Pad13): track 0.00 -> 10.2 mm
- net Net-(DRV2-Pad14): track 0.00 -> 9.94 mm
- net Net-(DRV2-Pad11): track 0.49 -> 10.4 mm
- net Net-(DRV1-Pad14): track 0.00 -> 9.72 mm
- net Net-(DRV1-Pad13): track 0.00 -> 9.50 mm
- net Net-(DRV1-Pad12): track 0.00 -> 9.28 mm
- net Net-(DRV1-Pad11): track 0.00 -> 9.05 mm

Commit message: Net
Parts:
- added REF**: 1pin, Connectors:1pin, F.Cu at (118.1, 110.5)
- added REF**: 1pin, Connectors:1pin, F.Cu at (118.1, 138.4)
- added REF**: 1pin, Connectors:1pin, F.Cu at (168.9, 153.7)
- added REF**: 1pin, Connectors:1pin, F.Cu at (168.9, 105.4)
Connections:
- DRV1 pad 1: (no net) -> Net-(DRV1-Pad1)
- DRV2 pad 1: (no net) -> Net-(DRV2-Pad1)
- U1 pad 10: (no net) -> Net-(U1-Pad10)
- U1 pad 11: (no net) -> Net-(U1-Pad11)
- U1 pad 12: (no net) -> Net-(U1-Pad12)
- U1 pad 14: (no net) -> Net-(U1-Pad14)
- U1 pad 15: (no net) -> Net-(U1-Pad15)
- U1 pad 16: Net-(DRV1-Pad7) -> Net-(U1-Pad16)
- U1 pad 17: Net-(DRV1-Pad8) -> Net-(U1-Pad17)
- U1 pad 18: (no net) -> Net-(U1-Pad18)
- U1 pad 19: (no net) -> Net-(U1-Pad19)
- U1 pad 2: (no net) -> Net-(U1-Pad2)
- U1 pad 21: (no net) -> Net-(U1-Pad21)
- U1 pad 23: (no net) -> Net-(U1-Pad23)
- U1 pad 24: (no net) -> Net-(U1-Pad24)
- U1 pad 26: (no net) -> Net-(U1-Pad26)
- U1 pad 27: (no net) -> Net-(U1-Pad27)
- U1 pad 28: (no net) -> Net-(U1-Pad28)
- U1 pad 29: (no net) -> Net-(U1-Pad29)
- U1 pad 3: (no net) -> Net-(U1-Pad3)
- U1 pad 30: (no net) -> Net-(DRV1-Pad7)
- U1 pad 31: (no net) -> Net-(DRV1-Pad8)
- U1 pad 33: (no net) -> Net-(U1-Pad33)
- U1 pad 35: (no net) -> Net-(U1-Pad35)
- U1 pad 38: (no net) -> Net-(U1-Pad38)
- U1 pad 4: (no net) -> Net-(U1-Pad4)
- U1 pad 5: (no net) -> Net-(U1-Pad5)
- U1 pad 7: (no net) -> Net-(U1-Pad7)
- U1 pad 8: (no net) -> Net-(U1-Pad8)
- U1 pad 9: (no net) -> Net-(U1-Pad9)
- U3 pad 5: (no net) -> Net-(U3-Pad5)
- U3 pad 6: (no net) -> Net-(U3-Pad6)
- U3 pad 7: (no net) -> Net-(U3-Pad7)
- U3 pad 8: (no net) -> Net-(U3-Pad8)
Routing:
- net Net-(DRV1-Pad7): track 0.00 -> 15.0 mm
- net Net-(DRV1-Pad8): track 0.00 -> 10.7 mm

Commit message: Gbert
Routing:
- net Net-(R1-Pad2): track 127.1 -> 123.2 mm
Changed lines of the file:
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@@
     (links 63)
     (no_connects 3)
-    (area 114.224999 91.364999 205.815001 162.635001)
+    (area 114.199999 91.339999 205.840001 162.660001)
     (thickness 1.6)
     (drawings 13)
-    (tracks 172)
+    (tracks 173)
     (zones 0)
     (modules 25)
@@
       (drillshape 0)
       (scaleselection 1)
-      (outputdirectory ""))
+      (outputdirectory output/))
   )
   (net 0 "")
@@
   (segment (start 127 148.59) (end 127 143.51) (width 0.25) (layer F.Cu) (net 21))
   (segment (start 125.73 149.86) (end 127 148.59) (width 0.25) (layer F.Cu) (net 21))
-  (segment (start 201.93 137.16) (end 203.2 137.16) (width 0.5) (layer F.Cu) (net 23))
-  (segment (start 129.54 138.43) (end 127 135.89) (width 0.5) (layer F.Cu) (net 23))
-  (segment (start 129.54 156.21) (end 129.54 138.43) (width 0.5) (layer F.Cu) (net 23))
-  (segment (start 132.08 158.75) (end 129.54 156.21) (width 0.5) (layer F.Cu) (net 23))
-  (segment (start 201.93 158.75) (end 132.08 158.75) (width 0.5) (layer F.Cu) (net 23))
-  (segment (start 203.2 157.48) (end 201.93 158.75) (width 0.5) (layer F.Cu) (net 23))
-  (segment (start 203.2 137.16) (end 203.2 157.48) (width 0.5) (layer F.Cu) (net 23))
+  (segment (start 201.93 137.16) (end 196.85 137.16) (width 0.5) (layer F.Cu) (net 23) (status 400000))
+  (segment (start 129.54 137.16) (end 127 134.62) (width 0.5) (layer F.Cu) (net 23) (status 800000))
+  (segment (start 129.54 157.48) (end 129.54 137.16) (width 0.5) (layer F.Cu) (net 23))
+  (segment (start 132.08 160.02) (end 129.54 157.48) (width 0.5) (layer F.Cu) (net 23))
+  (segment (start 186.69 160.02) (end 132.08 160.02) (width 0.5) (layer F.Cu) (net 23))
+  (segment (start 194.31 152.4) (end 186.69 160.02) (width 0.5) (layer F.Cu) (net 23))
+  (segment (start 194.31 139.7) (end 194.31 152.4) (width 0.5) (layer F.Cu) (net 23))
+  (segment (start 196.85 137.16) (end 194.31 139.7) (width 0.5) (layer F.Cu) (net 23))
   (segment (start 127 135.89) (end 127 134.62) (width 0.5) (layer F.Cu) (net 23))
   (segment (start 127 134.62) (end 127 138.43) (width 0.5) (layer F.Cu) (net 23))
