File: KiCad/_autosave-robot_blance.kicad_pcb (KiCad board)
At the start: 2 copper layers, 21 parts, among them J1 Bat, J10 CONN_01X02, J11 CONN_01X03, J2 CONN_01X04, J3 CONN_01X04, J4 CONN_01X02, J5 CONN_01X02, J6 CONN_01X02, J7 CONN_01X03, J8 CONN_01X02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

Commit message: Net
Other:
- net class Default: trace_width 0.25 -> 1
Changed lines of the file:
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@@
   )
   (setup
-    (last_trace_width 0.25)
+    (last_trace_width 1)
     (trace_clearance 0.2)
     (zone_clearance 0.508)
@@
   (net_class Default "This is the default net class."
     (clearance 0.2)
-    (trace_width 0.25)
+    (trace_width 1)
     (via_dia 0.6)
     (via_drill 0.4)
@@
     (polygon
       (pts
-        (xy 205.74 162.56) (xy 114.3 162.56) (xy 114.3 91.44) (xy 205.74 91.44) (xy 205.74 162.56)
+        (xy 205.74 162.56) (xy 114.3 162.56) (xy 114.3 91.44) (xy 205.74 91.44)
       )
     )
