File: KiCad/robot_blance.sch (KiCad schematic (older format))
At the start: 6 parts, among them J1 Bat, U1 Esp32Dev, U2 MP1584, U3 MPU6050

Commit message: Servo
Parts:
- added C1, C2: CP1, symbol CP1
- added D1: D, Diodes_THT:D_DO-41_SOD81_P7.62mm_Horizontal, symbol D
- added J10, J4, J5, J6, J8, J9: CONN_01X02, Connectors:PINHEAD1-2, symbol CONN_01X02
- added J11, J7: CONN_01X03, Connectors:PINHEAD1-3, symbol CONN_01X03
- added J2, J3: CONN_01X04, Connectors:Grove_1x04, symbol CONN_01X04
- added R1, R2: R, Resistors_THT:R_Axial_DIN0204_L3.6mm_D1.6mm_P5.08mm_Horizontal, symbol R
Connections:
- net +12V: now also D1.1 (K); no longer U2.1
- net GND: now also R2.1
- net at U1.1 (5v), U2.4, U3.1 (Vcc): now also DRV1.10 (FAULT), DRV2.10 (FAULT), J11.2 (P2), J4.2 (P2), J5.2 (P2), J6.2 (P2), J7.2 (P2)
- net at U1.13 (GPIO32): now also R1.2, R2.2
- net at U1.16 (GPIO39): now also DRV1.7 (STEP)
- net at U1.17 (GPIO36): now also DRV1.8 (DIR)
- net at U1.22 (GPIO22): now also U3.3 (Scl)
- net at U1.25 (GPIO21): now also U3.4 (Sda)
- net at U1.32 (GPIO4): now also DRV2.8 (DIR)
- net at U1.34 (GPIO2): now also DRV2.7 (STEP)
- net at U1.36 (GPIO8): now also J11.1 (P1)
- net at U1.37 (GPIO7): now also J7.1 (P1)
- net at DRV1.11 (A2): now also J2.4 (P4)
- net at DRV1.12 (A1): now also J2.3 (P3)
- net at DRV1.13 (B1): now also J2.2 (P2)
- net at DRV1.14 (B2): now also J2.1 (P1)
- net at DRV1.15 (GND): now also DRV1.9 (GND), DRV2.15 (GND), DRV2.9 (GND), U1.6 (GND), U2.3, C1.2, C2.2, J11.3 (P3), J7.3 (P3)
- net at DRV1.16 (VMOT): now also DRV2.16 (VMOT), U2.1, C1.1, C2.1, D1.2 (A), R1.1
- net at DRV1.2 (MO): now also J4.1 (P1)
- net at DRV1.3 (M1): now also J5.1 (P1)
- net at DRV1.4 (M2): now also J6.1 (P1)
- net at DRV1.5 (RESET): now also DRV1.6 (SLEEP)
- net at DRV2.11 (A2): now also J3.4 (P4)
- net at DRV2.12 (A1): now also J3.3 (P3)
- net at DRV2.13 (B1): now also J3.2 (P2)
- net at DRV2.14 (B2): now also J3.1 (P1)
- net at DRV2.2 (MO): now also J8.1 (P1)
- net at DRV2.3 (M1): now also J9.1 (P1)
- net at DRV2.4 (M2): now also J10.1 (P1)
- net at DRV2.5 (RESET): now also DRV2.6 (SLEEP)
- new net: J10.2 (P2), J8.2 (P2), J9.2 (P2)
- now unconnected: U2.3, U3.2 (Gnd)
Other:
- moved on the sheet: DRV1, DRV2, J1, U1, U2, U3

Commit message: Router
Parts:
- C1, C2: footprint (none) -> Capacitors_THT:CP_Radial_D10.0mm_P3.50mm
- D1: footprint Diodes_THT:D_DO-41_SOD81_P7.62mm_Horizontal -> Diodes_THT:D_DO-41_SOD81_P5.08mm_Vertical_AnodeUp
Connections:
- net GND: now also C1.2, C2.2, DRV1.15 (GND), DRV1.9 (GND), DRV2.15 (GND), DRV2.9 (GND), J11.3 (P3), J7.3 (P3), U1.6 (GND), U2.3, U3.2 (Gnd)
Changed lines of the file:
@@
 $EndComp
 $Comp
-L +12V #PWR2
+L +12V #PWR01
 U 1 1 5A58AA9D
 P 2300 2800
-F 0 "#PWR2" H 2300 2650 50  0001 C CNN
+F 0 "#PWR01" H 2300 2650 50  0001 C CNN
 F 1 "+12V" H 2300 2940 50  0000 C CNN
 F 2 "" H 2300 2800 50  0001 C CNN
@@
 $EndComp
 $Comp
-L GND #PWR1
+L GND #PWR02
 U 1 1 5A58AB89
 P 2300 2200
-F 0 "#PWR1" H 2300 1950 50  0001 C CNN
+F 0 "#PWR02" H 2300 1950 50  0001 C CNN
 F 1 "GND" H 2300 2050 50  0000 C CNN
 F 2 "" H 2300 2200 50  0001 C CNN
@@
 F 0 "D1" H 2600 2650 50  0000 C CNN
 F 1 "D" H 2600 2450 50  0000 C CNN
-F 2 "Diodes_THT:D_DO-41_SOD81_P7.62mm_Horizontal" H 2600 2550 50  0001 C CNN
+F 2 "Diodes_THT:D_DO-41_SOD81_P5.08mm_Vertical_AnodeUp" H 2600 2550 50  0001 C CNN
 F 3 "" H 2600 2550 50  0001 C CNN
 	1    2600 2550
@@
 F 0 "C1" H 7175 4750 50  0000 L CNN
 F 1 "CP1" H 7175 4550 50  0000 L CNN
-F 2 "" H 7150 4650 50  0001 C CNN
+F 2 "Capacitors_THT:CP_Radial_D10.0mm_P3.50mm" H 7150 4650 50  0001 C CNN
 F 3 "" H 7150 4650 50  0001 C CNN
 	1    7150 4650
@@
 F 0 "C2" H 9275 4750 50  0000 L CNN
 F 1 "CP1" H 9275 4550 50  0000 L CNN
-F 2 "" H 9250 4650 50  0001 C CNN
+F 2 "Capacitors_THT:CP_Radial_D10.0mm_P3.50mm" H 9250 4650 50  0001 C CNN
 F 3 "" H 9250 4650 50  0001 C CNN
 	1    9250 4650
@@
 $EndComp
 Wire Wire Line
-	6350 3550 6050 3550
-Wire Wire Line
-	6050 3550 6050 2250
-Wire Wire Line
-	6050 2250 4100 2250
-Wire Wire Line
 	6350 4050 5900 4050
 Wire Wire Line
@@
 Wire Wire Line
 	8400 3400 8400 4200
-Wire Wire Line
-	8650 3300 8350 3300
-Wire Wire Line
-	8350 3300 8350 2050
-Wire Wire Line
-	8350 2050 5800 2050
-Wire Wire Line
-	5800 2250 5800 1800
 Wire Wire Line
 	8400 4200 4100 4200
@@
 	8150 2750 8000 2750
 Wire Wire Line
-	8800 5300 8800 5600
-Wire Wire Line
-	9750 5600 6700 5600
-Wire Wire Line
-	6700 5300 6700 5800
-Wire Wire Line
-	5800 1800 9750 1800
-Wire Wire Line
-	9750 1800 9750 5600
-Connection ~ 8800 5600
-Wire Wire Line
 	4100 5500 9050 5500
 Wire Wire Line
@@
 Wire Wire Line
 	9100 4700 9100 4800
-Wire Wire Line
-	9100 4800 9750 4800
-Wire Wire Line
-	7150 4800 7150 5850
-Wire Wire Line
-	7150 5850 9250 5850
-Wire Wire Line
-	9250 5850 9250 4800
-Connection ~ 9750 4800
 Connection ~ 9250 4800
 Wire Wire Line
@@
 Connection ~ 5800 2750
 Wire Wire Line
-	4100 2750 4100 4200
+	4100 4200 4100 2650
 Wire Wire Line
 	9050 5500 9050 5200
@@
 	7150 4500 7150 4350
 Wire Wire Line
-	3250 4350 3250 2750
+	3250 4350 3250 2650
 Connection ~ 7150 4350
 Wire Wire Line
@@
 $EndComp
 Wire Wire Line
-	6100 6000 6100 5800
-Wire Wire Line
-	6100 5800 6700 5800
-Connection ~ 6700 5600
-Wire Wire Line
 	6200 6000 6200 5900
 Wire Wire Line
 	6200 5900 6850 5900
-Wire Wire Line
-	8200 6000 8200 5600
-Connection ~ 8200 5600
 Wire Wire Line
 	8300 6000 8300 5500
@@
 Wire Wire Line
 	10100 3850 8000 3850
+Connection ~ 3250 2750
+Wire Wire Line
+	3250 2350 3250 2250
+Wire Wire Line
+	4100 2250 4100 2350
+Connection ~ 4100 2750
+$Comp
+L GND #PWR?
+U 1 1 5A5C8868
+P 6150 3550
+F 0 "#PWR?" H 6150 3300 50  0001 C CNN
+F 1 "GND" H 6150 3400 50  0000 C CNN
+F 2 "" H 6150 3550 50  0001 C CNN
+F 3 "" H 6150 3550 50  0001 C CNN
+	1    6150 3550
+	1    0    0    -1
+$EndComp
+Wire Wire Line
+	6350 3550 6150 3550
+$Comp
+L GND #PWR?
+U 1 1 5A5C8BC3
+P 4250 2250
+F 0 "#PWR?" H 4250 2000 50  0001 C CNN
+F 1 "GND" H 4250 2100 50  0000 C CNN
+F 2 "" H 4250 2250 50  0001 C CNN
+F 3 "" H 4250 2250 50  0001 C CNN
+	1    4250 2250
+	1    0    0    -1
+$EndComp
+Wire Wire Line
+	4100 2250 4250 2250
+$Comp
+L GND #PWR?
+U 1 1 5A5C9A7E
+P 8500 3300
+F 0 "#PWR?" H 8500 3050 50  0001 C CNN
+F 1 "GND" H 8500 3150 50  0000 C CNN
+F 2 "" H 8500 3300 50  0001 C CNN
+F 3 "" H 8500 3300 50  0001 C CNN
+	1    8500 3300
+	1    0    0    -1
+$EndComp
+Wire Wire Line
+	8650 3300 8500 3300
+Wire Wire Line
+	9100 4800 9750 4800
+$Comp
+L GND #PWR?
+U 1 1 5A5CA562
+P 9750 4800
+F 0 "#PWR?" H 9750 4550 50  0001 C CNN
+F 1 "GND" H 9750 4650 50  0000 C CNN
+F 2 "" H 9750 4800 50  0001 C CNN
+F 3 "" H 9750 4800 50  0001 C CNN
+	1    9750 4800
+	1    0    0    -1
+$EndComp
+$Comp
+L GND #PWR?
+U 1 1 5A5CA6D7
+P 8950 5300
+F 0 "#PWR?" H 8950 5050 50  0001 C CNN
+F 1 "GND" H 8950 5150 50  0000 C CNN
+F 2 "" H 8950 5300 50  0001 C CNN
+F 3 "" H 8950 5300 50  0001 C CNN
+	1    8950 5300
+	1    0    0    -1
+$EndComp
+Wire Wire Line
+	8950 5300 8800 5300
+$Comp
+L GND #PWR?
+U 1 1 5A5CA943
+P 8000 6000
+F 0 "#PWR?" H 8000 5750 50  0001 C CNN
+F 1 "GND" H 8000 5850 50  0000 C CNN
+F 2 "" H 8000 6000 50  0001 C CNN
+F 3 "" H 8000 6000 50  0001 C CNN
+	1    8000 6000
+	1    0    0    -1
+$EndComp
+Wire Wire Line
+	8000 6000 8200 6000
+$Comp
+L GND #PWR?
+U 1 1 5A5CAB65
+P 6800 5300
+F 0 "#PWR?" H 6800 5050 50  0001 C CNN
+F 1 "GND" H 6800 5150 50  0000 C CNN
+F 2 "" H 6800 5300 50  0001 C CNN
+F 3 "" H 6800 5300 50  0001 C CNN
+	1    6800 5300
+	1    0    0    -1
+$EndComp
+Wire Wire Line
+	6700 5300 6800 5300
+$Comp
+L GND #PWR?
+U 1 1 5A5CAC52
+P 5950 6000
+F 0 "#PWR?" H 5950 5750 50  0001 C CNN
+F 1 "GND" H 5950 5850 50  0000 C CNN
+F 2 "" H 5950 6000 50  0001 C CNN
+F 3 "" H 5950 6000 50  0001 C CNN
+	1    5950 6000
+	1    0    0    -1
+$EndComp
+Wire Wire Line
+	5950 6000 6100 6000
+$Comp
+L GND #PWR?
+U 1 1 5A5CAFED
+P 7150 4950
+F 0 "#PWR?" H 7150 4700 50  0001 C CNN
+F 1 "GND" H 7150 4800 50  0000 C CNN
+F 2 "" H 7150 4950 50  0001 C CNN
+F 3 "" H 7150 4950 50  0001 C CNN
+	1    7150 4950
+	1    0    0    -1
+$EndComp
+Wire Wire Line
+	7150 4800 7150 4950
 $EndSCHEMATC

Commit message: router
Connections:
- net at DRV1.10 (FAULT), DRV2.10 (FAULT), J11.2 (P2)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: now also J10.2 (P2), J8.2 (P2), J9.2 (P2)
Changed lines of the file:
@@
 	7350 4500 7250 4500
 Wire Wire Line
-	7250 4500 7250 5100
+	7250 4500 7250 5500
 Wire Wire Line
 	7250 4800 7350 4800
@@
 Connection ~ 4100 2750
 $Comp
-L GND #PWR?
+L GND #PWR03
 U 1 1 5A5C8868
 P 6150 3550
-F 0 "#PWR?" H 6150 3300 50  0001 C CNN
+F 0 "#PWR03" H 6150 3300 50  0001 C CNN
 F 1 "GND" H 6150 3400 50  0000 C CNN
 F 2 "" H 6150 3550 50  0001 C CNN
@@
 	6350 3550 6150 3550
 $Comp
-L GND #PWR?
+L GND #PWR04
 U 1 1 5A5C8BC3
 P 4250 2250
-F 0 "#PWR?" H 4250 2000 50  0001 C CNN
+F 0 "#PWR04" H 4250 2000 50  0001 C CNN
 F 1 "GND" H 4250 2100 50  0000 C CNN
 F 2 "" H 4250 2250 50  0001 C CNN
@@
 	4100 2250 4250 2250
 $Comp
-L GND #PWR?
+L GND #PWR05
 U 1 1 5A5C9A7E
 P 8500 3300
-F 0 "#PWR?" H 8500 3050 50  0001 C CNN
+F 0 "#PWR05" H 8500 3050 50  0001 C CNN
 F 1 "GND" H 8500 3150 50  0000 C CNN
 F 2 "" H 8500 3300 50  0001 C CNN
@@
 	9100 4800 9750 4800
 $Comp
-L GND #PWR?
+L GND #PWR06
 U 1 1 5A5CA562
 P 9750 4800
-F 0 "#PWR?" H 9750 4550 50  0001 C CNN
+F 0 "#PWR06" H 9750 4550 50  0001 C CNN
 F 1 "GND" H 9750 4650 50  0000 C CNN
 F 2 "" H 9750 4800 50  0001 C CNN
@@
 $EndComp
 $Comp
-L GND #PWR?
+L GND #PWR07
 U 1 1 5A5CA6D7
 P 8950 5300
-F 0 "#PWR?" H 8950 5050 50  0001 C CNN
+F 0 "#PWR07" H 8950 5050 50  0001 C CNN
 F 1 "GND" H 8950 5150 50  0000 C CNN
 F 2 "" H 8950 5300 50  0001 C CNN
@@
 	8950 5300 8800 5300
 $Comp
-L GND #PWR?
+L GND #PWR08
 U 1 1 5A5CA943
 P 8000 6000
-F 0 "#PWR?" H 8000 5750 50  0001 C CNN
+F 0 "#PWR08" H 8000 5750 50  0001 C CNN
 F 1 "GND" H 8000 5850 50  0000 C CNN
 F 2 "" H 8000 6000 50  0001 C CNN
@@
 	8000 6000 8200 6000
 $Comp
-L GND #PWR?
+L GND #PWR09
 U 1 1 5A5CAB65
 P 6800 5300
-F 0 "#PWR?" H 6800 5050 50  0001 C CNN
+F 0 "#PWR09" H 6800 5050 50  0001 C CNN
 F 1 "GND" H 6800 5150 50  0000 C CNN
 F 2 "" H 6800 5300 50  0001 C CNN
@@
 	6700 5300 6800 5300
 $Comp
-L GND #PWR?
+L GND #PWR010
 U 1 1 5A5CAC52
 P 5950 6000
-F 0 "#PWR?" H 5950 5750 50  0001 C CNN
+F 0 "#PWR010" H 5950 5750 50  0001 C CNN
 F 1 "GND" H 5950 5850 50  0000 C CNN
 F 2 "" H 5950 6000 50  0001 C CNN
@@
 	5950 6000 6100 6000
 $Comp
-L GND #PWR?
+L GND #PWR011
 U 1 1 5A5CAFED
 P 7150 4950
-F 0 "#PWR?" H 7150 4700 50  0001 C CNN
+F 0 "#PWR011" H 7150 4700 50  0001 C CNN
 F 1 "GND" H 7150 4800 50  0000 C CNN
 F 2 "" H 7150 4950 50  0001 C CNN
@@
 Wire Wire Line
 	7150 4800 7150 4950
+Connection ~ 7250 5500
+Connection ~ 7250 5100
 $EndSCHEMATC

Commit message: Net
Connections:
- net +12V: now also C1.1, C2.1, DRV1.16 (VMOT), DRV2.16 (VMOT), U2.1
- net +5V: now reaches DRV1.10 (FAULT), DRV2.10 (FAULT), J10.2 (P2), J11.2 (P2), J4.2 (P2), J5.2 (P2), J6.2 (P2), J7.2 (P2), J8.2 (P2), J9.2 (P2), U1.1 (5v), U2.4, U3.1 (Vcc)
- new net: D1.2 (A), R1.1, U2.1
Changed lines of the file:
@@
 $EndComp
 Wire Wire Line
-	6350 4050 5900 4050
-Wire Wire Line
-	8650 3400 8400 3400
-Wire Wire Line
-	8400 3400 8400 4200
-Wire Wire Line
-	8400 4200 4100 4200
-Wire Wire Line
-	5900 4050 5900 2750
-Wire Wire Line
-	5900 2750 4100 2750
-Wire Wire Line
-	2300 2450 3150 2450
+	2300 2450 3050 2450
+Wire Wire Line
+	3050 2450 3150 2450
 Wire Wire Line
 	3150 2450 3150 2350
@@
 	2800 3100 2800 3250
 Wire Wire Line
-	2800 3250 3050 3250
+	2800 3250 2900 3250
+Wire Wire Line
+	2900 3250 3050 3250
 Wire Wire Line
 	3050 3250 3050 3100
 Wire Wire Line
-	2750 2550 3150 2550
+	2750 2550 2800 2550
+Wire Wire Line
+	2800 2550 3150 2550
 Wire Wire Line
 	2800 2550 2800 2800
@@
 	8150 2750 8000 2750
 Wire Wire Line
-	4100 5500 9050 5500
-Wire Wire Line
-	6850 5200 6850 5900
-Wire Wire Line
-	6850 5200 6700 5200
+	6700 5200 6900 5200
 Wire Wire Line
 	6700 4600 6700 4500
@@
 Wire Wire Line
 	8800 4500 9250 4500
+Wire Wire Line
+	9250 4500 9500 4500
 Wire Wire Line
 	8800 4700 9100 4700
@@
 Wire Wire Line
 	5000 2550 6350 2550
-Connection ~ 5800 2250
-Connection ~ 5800 2750
-Wire Wire Line
-	4100 4200 4100 2650
-Wire Wire Line
-	9050 5500 9050 5200
 Wire Wire Line
 	9050 5200 8800 5200
 Wire Wire Line
-	4100 5500 4100 4150
-Connection ~ 4100 4150
-Connection ~ 6850 5500
-Wire Wire Line
 	7700 5300 7500 5300
 Wire Wire Line
@@
 	7600 5200 7700 5200
 Wire Wire Line
-	9250 4500 9250 4350
-Wire Wire Line
-	9250 4350 3250 4350
-Wire Wire Line
-	7150 4500 7150 4350
-Wire Wire Line
-	3250 4350 3250 2650
-Connection ~ 7150 4350
-Wire Wire Line
 	5600 5100 5600 5000
 Wire Wire Line
@@
 	5300 4400 5100 4400
 Wire Wire Line
-	5100 4400 5100 5500
+	5100 4400 5100 4700
+Wire Wire Line
+	5100 4700 5100 5050
+Wire Wire Line
+	5100 5050 5100 5700
 Wire Wire Line
 	5100 4700 5300 4700
@@
 	5100 5050 5300 5050
 Connection ~ 5100 4700
-Connection ~ 5100 5500
 Connection ~ 5100 5050
 Wire Wire Line
@@
 	7350 4500 7250 4500
 Wire Wire Line
-	7250 4500 7250 5500
+	7250 4500 7250 4800
+Wire Wire Line
+	7250 4800 7250 5100
+Wire Wire Line
+	7250 5100 7250 5650
 Wire Wire Line
 	7250 4800 7350 4800
@@
 	6200 6000 6200 5900
 Wire Wire Line
-	6200 5900 6850 5900
-Wire Wire Line
-	8300 6000 8300 5500
-Connection ~ 8300 5500
-Wire Wire Line
 	6300 6000 6300 5950
 Wire Wire Line
@@
 Wire Wire Line
 	10100 3850 8000 3850
-Connection ~ 3250 2750
 Wire Wire Line
 	3250 2350 3250 2250
 Wire Wire Line
 	4100 2250 4100 2350
-Connection ~ 4100 2750
 $Comp
 L GND #PWR03
@@
 	8650 3300 8500 3300
 Wire Wire Line
-	9100 4800 9750 4800
+	9100 4800 9250 4800
+Wire Wire Line
+	9250 4800 9750 4800
 $Comp
 L GND #PWR06
@@
 Wire Wire Line
 	7150 4800 7150 4950
-Connection ~ 7250 5500
 Connection ~ 7250 5100
+$Comp
+L +12V #PWR?
+U 1 1 5A5F265E
+P 9500 4500
+F 0 "#PWR?" H 9500 4350 50  0001 C CNN
+F 1 "+12V" H 9500 4640 50  0000 C CNN
+F 2 "" H 9500 4500 50  0001 C CNN
+F 3 "" H 9500 4500 50  0001 C CNN
+	1    9500 4500
+	1    0    0    -1
+$EndComp
+Connection ~ 9250 4500
+$Comp
+L +12V #PWR?
+U 1 1 5A5F2A22
+P 7150 4450
+F 0 "#PWR?" H 7150 4300 50  0001 C CNN
+F 1 "+12V" H 7150 4590 50  0000 C CNN
+F 2 "" H 7150 4450 50  0001 C CNN
+F 3 "" H 7150 4450 50  0001 C CNN
+	1    7150 4450
+	1    0    0    -1
+$EndComp
+Wire Wire Line
+	7150 4500 7150 4450
+$Comp
+L +5V #PWR?
+U 1 1 5A5F374B
+P 6150 4050
+F 0 "#PWR?" H 6150 3900 50  0001 C CNN
+F 1 "+5V" H 6150 4190 50  0000 C CNN
+F 2 "" H 6150 4050 50  0001 C CNN
+F 3 "" H 6150 4050 50  0001 C CNN
+	1    6150 4050
+	1    0    0    -1
+$EndComp
+Wire Wire Line
+	6350 4050 6150 4050
+Wire Wire Line
+	4100 2650 4100 2750
+$Comp
+L +5V #PWR?
+U 1 1 5A5F3BEE
+P 4250 2750
+F 0 "#PWR?" H 4250 2600 50  0001 C CNN
+F 1 "+5V" H 4250 2890 50  0000 C CNN
+F 2 "" H 4250 2750 50  0001 C CNN
+F 3 "" H 4250 2750 50  0001 C CNN
+	1    4250 2750
+	1    0    0    -1
+$EndComp
+Wire Wire Line
+	4100 2750 4250 2750
+Wire Wire Line
+	3250 2650 3250 2900
+$Comp
+L +12V #PWR?
+U 1 1 5A5F3FA7
+P 3250 2900
+F 0 "#PWR?" H 3250 2750 50  0001 C CNN
+F 1 "+12V" H 3250 3040 50  0000 C CNN
+F 2 "" H 3250 2900 50  0001 C CNN
+F 3 "" H 3250 2900 50  0001 C CNN
+	1    3250 2900
+	1    0    0    1
+$EndComp
+$Comp
+L +5V #PWR?
+U 1 1 5A5F4789
+P 8650 3400
+F 0 "#PWR?" H 8650 3250 50  0001 C CNN
+F 1 "+5V" H 8650 3540 50  0000 C CNN
+F 2 "" H 8650 3400 50  0001 C CNN
+F 3 "" H 8650 3400 50  0001 C CNN
+	1    8650 3400
+	1    0    0    1
+$EndComp
+$Comp
+L +5V #PWR?
+U 1 1 5A5F4B3B
+P 5100 5700
+F 0 "#PWR?" H 5100 5550 50  0001 C CNN
+F 1 "+5V" H 5100 5840 50  0000 C CNN
+F 2 "" H 5100 5700 50  0001 C CNN
+F 3 "" H 5100 5700 50  0001 C CNN
+	1    5100 5700
+	1    0    0    1
+$EndComp
+$Comp
+L +5V #PWR?
+U 1 1 5A5F4F1C
+P 7250 5650
+F 0 "#PWR?" H 7250 5500 50  0001 C CNN
+F 1 "+5V" H 7250 5790 50  0000 C CNN
+F 2 "" H 7250 5650 50  0001 C CNN
+F 3 "" H 7250 5650 50  0001 C CNN
+	1    7250 5650
+	1    0    0    1
+$EndComp
+$Comp
+L +5V #PWR?
+U 1 1 5A5F5570
+P 6900 5200
+F 0 "#PWR?" H 6900 5050 50  0001 C CNN
+F 1 "+5V" H 6900 5340 50  0000 C CNN
+F 2 "" H 6900 5200 50  0001 C CNN
+F 3 "" H 6900 5200 50  0001 C CNN
+	1    6900 5200
+	1    0    0    1
+$EndComp
+$Comp
+L +5V #PWR?
+U 1 1 5A5F5807
+P 6200 5900
+F 0 "#PWR?" H 6200 5750 50  0001 C CNN
+F 1 "+5V" H 6200 6040 50  0000 C CNN
+F 2 "" H 6200 5900 50  0001 C CNN
+F 3 "" H 6200 5900 50  0001 C CNN
+	1    6200 5900
+	1    0    0    -1
+$EndComp
+$Comp
+L +5V #PWR?
+U 1 1 5A5F5989
+P 8300 5950
+F 0 "#PWR?" H 8300 5800 50  0001 C CNN
+F 1 "+5V" H 8300 6090 50  0000 C CNN
+F 2 "" H 8300 5950 50  0001 C CNN
+F 3 "" H 8300 5950 50  0001 C CNN
+	1    8300 5950
+	1    0    0    -1
+$EndComp
+Wire Wire Line
+	8300 6000 8300 5950
+$Comp
+L +5V #PWR?
+U 1 1 5A5F5B98
+P 9050 5200
+F 0 "#PWR?" H 9050 5050 50  0001 C CNN
+F 1 "+5V" H 9050 5340 50  0000 C CNN
+F 2 "" H 9050 5200 50  0001 C CNN
+F 3 "" H 9050 5200 50  0001 C CNN
+	1    9050 5200
+	1    0    0    1
+$EndComp
 $EndSCHEMATC

Commit message: Net
Connections:
- net GND: now also U1.20 (GND)
Changed lines of the file:
@@
 $EndComp
 Wire Wire Line
-	2300 2450 3050 2450
-Wire Wire Line
-	3050 2450 3150 2450
+	2300 2450 3150 2450
 Wire Wire Line
 	3150 2450 3150 2350
@@
 	2800 3100 2800 3250
 Wire Wire Line
-	2800 3250 2900 3250
-Wire Wire Line
-	2900 3250 3050 3250
+	2800 3250 3050 3250
 Wire Wire Line
 	3050 3250 3050 3100
 Wire Wire Line
-	2750 2550 2800 2550
-Wire Wire Line
-	2800 2550 3150 2550
+	2750 2550 3150 2550
 Wire Wire Line
 	2800 2550 2800 2800
@@
 	8800 4600 8800 4500
 Wire Wire Line
-	8800 4500 9250 4500
-Wire Wire Line
-	9250 4500 9500 4500
+	8800 4500 9500 4500
 Wire Wire Line
 	8800 4700 9100 4700
@@
 	5300 4400 5100 4400
 Wire Wire Line
-	5100 4400 5100 4700
-Wire Wire Line
-	5100 4700 5100 5050
-Wire Wire Line
-	5100 5050 5100 5700
+	5100 4400 5100 5700
 Wire Wire Line
 	5100 4700 5300 4700
@@
 	7350 4500 7250 4500
 Wire Wire Line
-	7250 4500 7250 4800
-Wire Wire Line
-	7250 4800 7250 5100
-Wire Wire Line
-	7250 5100 7250 5650
+	7250 4500 7250 5650
 Wire Wire Line
 	7250 4800 7350 4800
@@
 	8650 3300 8500 3300
 Wire Wire Line
-	9100 4800 9250 4800
-Wire Wire Line
-	9250 4800 9750 4800
+	9100 4800 9750 4800
 $Comp
 L GND #PWR06
@@
 Connection ~ 7250 5100
 $Comp
-L +12V #PWR?
+L +12V #PWR012
 U 1 1 5A5F265E
 P 9500 4500
-F 0 "#PWR?" H 9500 4350 50  0001 C CNN
+F 0 "#PWR012" H 9500 4350 50  0001 C CNN
 F 1 "+12V" H 9500 4640 50  0000 C CNN
 F 2 "" H 9500 4500 50  0001 C CNN
@@
 Connection ~ 9250 4500
 $Comp
-L +12V #PWR?
+L +12V #PWR013
 U 1 1 5A5F2A22
 P 7150 4450
-F 0 "#PWR?" H 7150 4300 50  0001 C CNN
+F 0 "#PWR013" H 7150 4300 50  0001 C CNN
 F 1 "+12V" H 7150 4590 50  0000 C CNN
 F 2 "" H 7150 4450 50  0001 C CNN
@@
 	7150 4500 7150 4450
 $Comp
-L +5V #PWR?
+L +5V #PWR014
 U 1 1 5A5F374B
 P 6150 4050
-F 0 "#PWR?" H 6150 3900 50  0001 C CNN
+F 0 "#PWR014" H 6150 3900 50  0001 C CNN
 F 1 "+5V" H 6150 4190 50  0000 C CNN
 F 2 "" H 6150 4050 50  0001 C CNN
@@
 	4100 2650 4100 2750
 $Comp
-L +5V #PWR?
+L +5V #PWR015
 U 1 1 5A5F3BEE
 P 4250 2750
-F 0 "#PWR?" H 4250 2600 50  0001 C CNN
+F 0 "#PWR015" H 4250 2600 50  0001 C CNN
 F 1 "+5V" H 4250 2890 50  0000 C CNN
 F 2 "" H 4250 2750 50  0001 C CNN
@@
 	3250 2650 3250 2900
 $Comp
-L +12V #PWR?
+L +12V #PWR016
 U 1 1 5A5F3FA7
 P 3250 2900
-F 0 "#PWR?" H 3250 2750 50  0001 C CNN
+F 0 "#PWR016" H 3250 2750 50  0001 C CNN
 F 1 "+12V" H 3250 3040 50  0000 C CNN
 F 2 "" H 3250 2900 50  0001 C CNN
@@
 $EndComp
 $Comp
-L +5V #PWR?
+L +5V #PWR017
 U 1 1 5A5F4789
 P 8650 3400
-F 0 "#PWR?" H 8650 3250 50  0001 C CNN
+F 0 "#PWR017" H 8650 3250 50  0001 C CNN
 F 1 "+5V" H 8650 3540 50  0000 C CNN
 F 2 "" H 8650 3400 50  0001 C CNN
@@
 $EndComp
 $Comp
-L +5V #PWR?
+L +5V #PWR018
 U 1 1 5A5F4B3B
 P 5100 5700
-F 0 "#PWR?" H 5100 5550 50  0001 C CNN
+F 0 "#PWR018" H 5100 5550 50  0001 C CNN
 F 1 "+5V" H 5100 5840 50  0000 C CNN
 F 2 "" H 5100 5700 50  0001 C CNN
@@
 $EndComp
 $Comp
-L +5V #PWR?
+L +5V #PWR019
 U 1 1 5A5F4F1C
 P 7250 5650
-F 0 "#PWR?" H 7250 5500 50  0001 C CNN
+F 0 "#PWR019" H 7250 5500 50  0001 C CNN
 F 1 "+5V" H 7250 5790 50  0000 C CNN
 F 2 "" H 7250 5650 50  0001 C CNN
@@
 $EndComp
 $Comp
-L +5V #PWR?
+L +5V #PWR020
 U 1 1 5A5F5570
 P 6900 5200
-F 0 "#PWR?" H 6900 5050 50  0001 C CNN
+F 0 "#PWR020" H 6900 5050 50  0001 C CNN
 F 1 "+5V" H 6900 5340 50  0000 C CNN
 F 2 "" H 6900 5200 50  0001 C CNN
@@
 $EndComp
 $Comp
-L +5V #PWR?
+L +5V #PWR021
 U 1 1 5A5F5807
 P 6200 5900
-F 0 "#PWR?" H 6200 5750 50  0001 C CNN
+F 0 "#PWR021" H 6200 5750 50  0001 C CNN
 F 1 "+5V" H 6200 6040 50  0000 C CNN
 F 2 "" H 6200 5900 50  0001 C CNN
@@
 $EndComp
 $Comp
-L +5V #PWR?
+L +5V #PWR022
 U 1 1 5A5F5989
 P 8300 5950
-F 0 "#PWR?" H 8300 5800 50  0001 C CNN
+F 0 "#PWR022" H 8300 5800 50  0001 C CNN
 F 1 "+5V" H 8300 6090 50  0000 C CNN
 F 2 "" H 8300 5950 50  0001 C CNN
@@
 	8300 6000 8300 5950
 $Comp
-L +5V #PWR?
+L +5V #PWR023
 U 1 1 5A5F5B98
 P 9050 5200
-F 0 "#PWR?" H 9050 5050 50  0001 C CNN
+F 0 "#PWR023" H 9050 5050 50  0001 C CNN
 F 1 "+5V" H 9050 5340 50  0000 C CNN
 F 2 "" H 9050 5200 50  0001 C CNN
@@
 	1    0    0    1
 $EndComp
+$Comp
+L GND #PWR?
+U 1 1 5A5F66F7
+P 8200 2250
+F 0 "#PWR?" H 8200 2000 50  0001 C CNN
+F 1 "GND" H 8200 2100 50  0000 C CNN
+F 2 "" H 8200 2250 50  0001 C CNN
+F 3 "" H 8200 2250 50  0001 C CNN
+	1    8200 2250
+	1    0    0    1
+$EndComp
+Wire Wire Line
+	8000 2250 8200 2250
 $EndSCHEMATC

Commit message: Net
Connections:
- net +12V: no longer C1.1, C2.1, DRV1.16 (VMOT), DRV2.16 (VMOT), U2.1
- net at D1.2 (A), R1.1, U2.1: now also C1.1, C2.1, DRV1.16 (VMOT), DRV2.16 (VMOT)
Changed lines of the file:
@@
 	8800 4600 8800 4500
-Wire Wire Line
-	8800 4500 9500 4500
 Wire Wire Line
 	8800 4700 9100 4700
@@
 	7150 4800 7150 4950
 Connection ~ 7250 5100
-$Comp
-L +12V #PWR012
-U 1 1 5A5F265E
-P 9500 4500
-F 0 "#PWR012" H 9500 4350 50  0001 C CNN
-F 1 "+12V" H 9500 4640 50  0000 C CNN
-F 2 "" H 9500 4500 50  0001 C CNN
-F 3 "" H 9500 4500 50  0001 C CNN
-	1    9500 4500
-	1    0    0    -1
-$EndComp
-Connection ~ 9250 4500
-$Comp
-L +12V #PWR013
-U 1 1 5A5F2A22
-P 7150 4450
-F 0 "#PWR013" H 7150 4300 50  0001 C CNN
-F 1 "+12V" H 7150 4590 50  0000 C CNN
-F 2 "" H 7150 4450 50  0001 C CNN
-F 3 "" H 7150 4450 50  0001 C CNN
-	1    7150 4450
-	1    0    0    -1
-$EndComp
-Wire Wire Line
-	7150 4500 7150 4450
+Wire Wire Line
+	7150 4500 7150 4300
 $Comp
 L +5V #PWR014
@@
 Wire Wire Line
 	4100 2750 4250 2750
-Wire Wire Line
-	3250 2650 3250 2900
-$Comp
-L +12V #PWR016
-U 1 1 5A5F3FA7
-P 3250 2900
-F 0 "#PWR016" H 3250 2750 50  0001 C CNN
-F 1 "+12V" H 3250 3040 50  0000 C CNN
-F 2 "" H 3250 2900 50  0001 C CNN
-F 3 "" H 3250 2900 50  0001 C CNN
-	1    3250 2900
-	1    0    0    1
-$EndComp
 $Comp
 L +5V #PWR017
@@
 Wire Wire Line
 	8000 2250 8200 2250
+Wire Wire Line
+	3250 2650 3250 4300
+Wire Wire Line
+	3250 4300 9250 4300
+Connection ~ 3250 2750
+Wire Wire Line
+	8800 4500 9250 4500
+Wire Wire Line
+	9250 4500 9250 4300
+Connection ~ 7150 4300
 $EndSCHEMATC
