File: KiCad/robot_blance.sch (KiCad schematic (older format))
At the start: 21 parts, among them J1 Bat, J10 CONN_01X02, J11 CONN_01X03, J2 CONN_01X04, J3 CONN_01X04, J4 CONN_01X02, J5 CONN_01X02, J6 CONN_01X02, J7 CONN_01X03, J8 CONN_01X02, J9 CONN_01X02, U1 Esp32Dev, U2 MP1584, U3 MPU6050

Commit message: Net
Connections:
- net at U1.16 (GPIO39): no longer DRV1.7 (STEP)
- net at U1.17 (GPIO36): no longer DRV1.8 (DIR)
- net at U1.30 (GPIO17): now also DRV1.7 (STEP)
- net at U1.31 (GPIO16): now also DRV1.8 (DIR)
Changed lines of the file:
@@
 	4900 5300 5600 5300
 Wire Wire Line
-	4900 2450 4900 5300
-Wire Wire Line
-	4900 2450 6350 2450
-Wire Wire Line
-	5600 5200 5000 5200
-Wire Wire Line
-	5000 5200 5000 2550
-Wire Wire Line
-	5000 2550 6350 2550
+	4900 1800 4900 5300
+Wire Wire Line
+	5000 5200 5600 5200
+Wire Wire Line
+	5000 1700 5000 5200
 Wire Wire Line
 	9050 5200 8800 5200
@@
 	9250 4500 9250 4300
 Connection ~ 7150 4300
+Wire Wire Line
+	4900 1800 8300 1800
+Wire Wire Line
+	8300 1800 8300 3350
+Wire Wire Line
+	8300 3350 8000 3350
+Wire Wire Line
+	5000 1700 8400 1700
+Wire Wire Line
+	8400 1700 8400 3250
+Wire Wire Line
+	8400 3250 8000 3250
 $EndSCHEMATC
